File: BigAssTKL.kicad_pcb (KiCad board)
At the start: 2 copper layers, 345 x 122 mm, 180 parts, among them J1 KEYSWITCH-PLAIN-MX-1U, K1 KEYSWITCH-PLAIN-MX-1U, M1 KEYSWITCH-PLAIN-MX-1U, P1 KEYSWITCH-PLAIN-MX-1U, Q1 KEYSWITCH-PLAIN-MX-1U, T1 KEYSWITCH-PLAIN-MX-1U, U1 KEYSWITCH-PLAIN-MX-1U, X1 KEYSWITCH-PLAIN-MX-1U, Y1 KEYSWITCH-PLAIN-MX-1U

Commit message: Add files via upload
Parts:
- removed ENTERTOP1: KEYSWITCH-PLAIN-MX-1U, Button_Switch_Keyboard:SW_Cherry_MX_1.50u_PCB
Other:
- outline, holes or cut-outs redrawn

Commit message: Add files via upload
Parts:
- removed DZ: , Diode_SMD:D_SOD-123_
- added REF**: D_SOD-123_, Diode_SMD:D_SOD-123_, B.Cu at (288.4, 148.9)
- D0, D1, D2, D3, D4, D5, D6, D7, D8, D9, DA1, DALT1, DALT2, DB1, DBACKSLASH1, DBACKSPACE1, DC1, DCAPSLOCK1, DCOMMA1, DCTRL1, DCTRL2, DD1, DDASH1, DDELETE1, DDOWN1, DE1, DEND1, DEQUAL1, DESC1, DF1, DF10, DF11, DF13, DF2, DF3, DF4, DF5, DF6, DF7, DF8, DF9, DFN1, DG1, DGRAVE1, DH1, DHOME1, DI1, DINSERT1, DJ1, DK1, DL1, DLBRACKET1, DLEFT1, DM1, DMENU1, DN1, DO1, DP1, DPAUSE1, DPERIOD1, DPGDN1, DPGUP1, DPRTSC1, DQ1, DQUOTE1, DR1, DRBRACKET1, DRIGHT1, DS1, DSCROLLLOCK1, DSEMICOLON1, DSHIFT1, DSHIFT2, DSLASH1, DSPACE1, DT1, DTAB1, DU1, DUP1, DV1, DW1, DWIN1, DX1, DY1, DZ1: moved to B.Cu
- DF12: renamed from DF; moved to B.Cu
- moved MCU 60.4 mm to (235.4, 94.4)
- moved DPRTSC1 1.40 mm to (328.1, 81.5)
- moved DINSERT1 1.40 mm to (328.0, 109.5)
- moved DDELETE1 0.20 mm to (328.0, 129.7)
- turned DPGDN1 to 90 degrees
- turned DPGUP1 to 90 degrees
Routing:
- net (no net): track 2931.2 -> 2651.2 mm, vias 10 -> 12
- net Net-(DF4-PadA): track 258.8 -> 371.8 mm
- net Net-(DF11-PadA): track 108.8 -> 215.9 mm
- net Net-(DF5-PadA): track 207.3 -> 310.7 mm
- net Net-(DZ1-PadA): track 326.4 -> 238.8 mm
- net Net-(DF13-PadA): track 175.6 -> 251.8 mm
- net Net-(DF12-PadA): track 129.7 -> 205.5 mm
- net Net-(DF3-PadA): track 146.3 -> 218.8 mm
- net Net-(DF2-PadA): track 174.4 -> 245.6 mm
- net Net-(DD1-PadA): track 276.4 -> 211.9 mm
- net Net-(DDASH1-PadA): track 173.6 -> 112.1 mm
- net Net-(DC1-PadA): track 178.7 -> 118.9 mm
- net Net-(DF10-PadA): track 121.7 -> 176.4 mm
- net Net-(DF1-PadA): track 313.2 -> 258.7 mm
- net Net-(D2-PadA): track 269.9 -> 215.9 mm, vias 1 -> 0
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- removed copper zone on B.Cu, net (none)
- removed copper zone on F.Cu, net (none)
Other:
- board size 345 x 122 mm -> 348 x 123.6 mm
